Commit message: -

File: src/hector_gazebo/assets/models/xacro/arm.xacro (robot description, xacro)
@@ -25,10 +25,10 @@
             <xacro:if value="${(mirror_dae == True)}">
             <geometry>
-                <mesh filename="file://$(find hector_assets)/models/meshes/hector_arm/ShoulderYaw_L.stl" scale="1 1 1"/>
+                <mesh filename="file://$(find hector_gazebo)/assets/models/meshes/hector_arm/ShoulderYaw_L.stl" scale="1 1 1"/>
             </geometry>
             </xacro:if>
             <xacro:if value="${(mirror_dae == False)}">
             <geometry>
-                <mesh filename="file://$(find hector_assets)/models/meshes/hector_arm/ShoulderYaw_R.stl" scale="1 1 1"/>
+                <mesh filename="file://$(find hector_gazebo)/assets/models/meshes/hector_arm/ShoulderYaw_R.stl" scale="1 1 1"/>
             </geometry>
             </xacro:if>
@@ -68,10 +68,10 @@
             <xacro:if value="${(mirror_dae == True)}">
             <geometry>
-                <mesh filename="file://$(find hector_assets)/models/meshes/hector_arm/ShoulderPitch_L.stl" scale="1 1 1"/>
+                <mesh filename="file://$(find hector_gazebo)/assets/models/meshes/hector_arm/ShoulderPitch_L.stl" scale="1 1 1"/>
             </geometry>
             </xacro:if>
             <xacro:if value="${(mirror_dae == False)}">
             <geometry>
-                <mesh filename="file://$(find hector_assets)/models/meshes/hector_arm/ShoulderPitch_R.stl" scale="1 1 1"/>
+                <mesh filename="file://$(find hector_gazebo)/assets/models/meshes/hector_arm/ShoulderPitch_R.stl" scale="1 1 1"/>
             </geometry>
             </xacro:if>
@@ -111,10 +111,10 @@
             <xacro:if value="${(mirror_dae == True)}">
             <geometry>
-                <mesh filename="file://$(find hector_assets)/models/meshes/hector_arm/UpperArmRoll_L.stl" scale="1 1 1"/>
+                <mesh filename="file://$(find hector_gazebo)/assets/models/meshes/hector_arm/UpperArmRoll_L.stl" scale="1 1 1"/>
             </geometry>
             </xacro:if>
             <xacro:if value="${(mirror_dae == False)}">
             <geometry>
-                <mesh filename="file://$(find hector_assets)/models/meshes/hector_arm/UpperArmRoll_R.stl" scale="1 1 1"/>
+                <mesh filename="file://$(find hector_gazebo)/assets/models/meshes/hector_arm/UpperArmRoll_R.stl" scale="1 1 1"/>
             </geometry>
             </xacro:if>
@@ -148,5 +148,5 @@
             <origin rpy="0 0 0" xyz="0 0 0"/>
             <geometry>
-                <mesh filename="file://$(find hector_assets)/models/meshes/hector_arm/ForeArmPitch.stl" scale="1 1 1"/>
+                <mesh filename="file://$(find hector_gazebo)/assets/models/meshes/hector_arm/ForeArmPitch.stl" scale="1 1 1"/>
             </geometry>
             <material name="grey"/>

File: src/hector_gazebo/assets/models/xacro/body.xacro (robot description, xacro)
@@ -24,5 +24,5 @@
             <origin rpy="0 0 0" xyz="0 0 0"/>
             <geometry>
-                <mesh filename="file://$(find hector_assets)/models/meshes/body.stl" scale="1 1 1"/>
+                <mesh filename="file://$(find hector_gazebo)/assets/models/meshes/body.stl" scale="1 1 1"/>
             </geometry>
             <material name="black"/>
@@ -83,5 +83,5 @@
             <origin rpy="0 0 0" xyz="0 0 0"/>
                 <geometry>
-                    <mesh filename="file://$(find hector_assets)/models/meshes/Head.STL" scale="0.001 0.001 0.001"/>
+                    <mesh filename="file://$(find hector_gazebo)/assets/models/meshes/Head.STL" scale="0.001 0.001 0.001"/>
                 </geometry>
             <material name="black"/>
@@ -109,5 +109,5 @@
             <origin rpy="0 0 0" xyz="0 0 0"/>
                 <geometry>
-                    <mesh filename="file://$(find hector_assets)/models/meshes/NUC_backpack.STL" scale="1 1 1"/>
+                    <mesh filename="file://$(find hector_gazebo)/assets/models/meshes/NUC_backpack.STL" scale="1 1 1"/>
                 </geometry>
             <material name="black"/>

File: src/hector_gazebo/assets/models/xacro/hardware.xacro (robot description, xacro)
@@ -207,12 +207,6 @@
         <plugin filename="libgazebo_ros2_control.so" name="gazebo_ros2_control">
           <robot_sim_type>gazebo_ros2_control/GazeboSystem</robot_sim_type>
-        <parameters>$(find hector_assets)/config/hector_controller_config.yaml</parameters>
+        <parameters>$(find hector_gazebo)/assets/config/hector_controller_config.yaml</parameters>
         </plugin>
     </gazebo>
-    <!-- <gazebo>
-      <plugin name="joint_state_publisher" filename="libgazebo_ros_joint_state_publisher.so">
-        <robotNamespace>/</robotNamespace>
-        <joint_name>L_hip_roll_joint</joint_name>
-      </plugin>
-    </gazebo>     -->
 </robot>

File: src/hector_gazebo/assets/models/xacro/leg.xacro (robot description, xacro)
@@ -1,5 +1,5 @@
 <?xml version="1.0"?>
 <robot xmlns:xacro="http://www.ros.org/wiki/xacro">
-    <!-- <xacro:include filename="$(find hector_assets)/models/xacro/transmission.xacro"/> -->
+    <!-- <xacro:include filename="$(find hector_gazebo)/assets/models/xacro/transmission.xacro"/> -->
     <xacro:macro name="leg" params="name mirror mirror_dae  *origin">
         <joint name="${name}_hip_yaw_joint" type="revolute">
@@ -21,10 +21,10 @@
                 <xacro:if value="${(mirror_dae == True)}">
                     <geometry>
-                        <mesh filename="file://$(find hector_assets)/models/meshes/R_hip_yaw.STL" scale="1 1 1"/>
-                    </geometry>
-                </xacro:if>
-                <xacro:if value="${(mirror_dae == False)}">
-                   <geometry>
-                        <mesh filename="file://$(find hector_assets)/models/meshes/L_hip_yaw.STL" scale="1 1 1"/>
+                        <mesh filename="file://$(find hector_gazebo)/assets/models/meshes/R_hip_yaw.STL" scale="1 1 1"/>
+                    </geometry>
+                </xacro:if>
+                <xacro:if value="${(mirror_dae == False)}">
+                   <geometry>
+                        <mesh filename="file://$(find hector_gazebo)/assets/models/meshes/L_hip_yaw.STL" scale="1 1 1"/>
                     </geometry>
                 </xacro:if>
@@ -86,10 +86,10 @@
                 <xacro:if value="${(mirror_dae == True)}">
                     <geometry>
-                        <mesh filename="file://$(find hector_assets)/models/meshes/R_hip_roll.STL" scale="1 1 1"/>
-                    </geometry>
-                </xacro:if>
-                <xacro:if value="${(mirror_dae == False)}">
-                   <geometry>
-                        <mesh filename="file://$(find hector_assets)/models/meshes/L_hip_roll.STL" scale="1 1 1"/>
+                        <mesh filename="file://$(find hector_gazebo)/assets/models/meshes/R_hip_roll.STL" scale="1 1 1"/>
+                    </geometry>
+                </xacro:if>
+                <xacro:if value="${(mirror_dae == False)}">
+                   <geometry>
+                        <mesh filename="file://$(find hector_gazebo)/assets/models/meshes/L_hip_roll.STL" scale="1 1 1"/>
                     </geometry>
                 </xacro:if>
@@ -152,10 +152,10 @@
                 <xacro:if value="${(mirror_dae == True)}">
                     <geometry>
-                        <mesh filename="file://$(find hector_assets)/models/meshes/hip_pitch_combined_R2.stl" scale="1 1 1"/>
-                    </geometry>
-                </xacro:if>
-                <xacro:if value="${(mirror_dae == False)}">
-                   <geometry>
-                        <mesh filename="file://$(find hector_assets)/models/meshes/hip_pitch_combined_L2.stl" scale="1 1 1"/>
+                        <mesh filename="file://$(find hector_gazebo)/assets/models/meshes/hip_pitch_combined_R2.stl" scale="1 1 1"/>
+                    </geometry>
+                </xacro:if>
+                <xacro:if value="${(mirror_dae == False)}">
+                   <geometry>
+                        <mesh filename="file://$(find hector_gazebo)/assets/models/meshes/hip_pitch_combined_L2.stl" scale="1 1 1"/>
                     </geometry>
                 </xacro:if>
@@ -234,10 +234,10 @@
                 <xacro:if value="${(mirror_dae == True)}">
                     <geometry>
-                        <mesh filename="file://$(find hector_assets)/models/meshes/knee_combined_R.stl" scale="1 1 1"/>
-                    </geometry>
-                </xacro:if>
-                <xacro:if value="${(mirror_dae == False)}">
-                   <geometry>
-                        <mesh filename="file://$(find hector_assets)/models/meshes/knee_combined_L.stl" scale="1 1 1"/>
+                        <mesh filename="file://$(find hector_gazebo)/assets/models/meshes/knee_combined_R.stl" scale="1 1 1"/>
+                    </geometry>
+                </xacro:if>
+                <xacro:if value="${(mirror_dae == False)}">
+                   <geometry>
+                        <mesh filename="file://$(find hector_gazebo)/assets/models/meshes/knee_combined_L.stl" scale="1 1 1"/>
                     </geometry>
                 </xacro:if>
@@ -272,10 +272,10 @@
                 <xacro:if value="${(mirror_dae == True)}">
                     <geometry>
-                        <mesh filename="file://$(find hector_assets)/models/meshes/foot_R2.stl" scale="1 1 1"/>
-                    </geometry>
-                </xacro:if>
-                <xacro:if value="${(mirror_dae == False)}">
-                   <geometry>
-                        <mesh filename="file://$(find hector_assets)/models/meshes/foot_L2.stl" scale="1 1 1"/>
+                        <mesh filename="file://$(find hector_gazebo)/assets/models/meshes/foot_R2.stl" scale="1 1 1"/>
+                    </geometry>
+                </xacro:if>
+                <xacro:if value="${(mirror_dae == False)}">
+                   <geometry>
+                        <mesh filename="file://$(find hector_gazebo)/assets/models/meshes/foot_L2.stl" scale="1 1 1"/>
                     </geometry>
                 </xacro:if>

File: src/hector_gazebo/assets/models/xacro/robot.xacro (robot description, xacro)
@@ -3,10 +3,10 @@
 <robot name="hector_v2" xmlns:xacro="http://www.ros.org/wiki/xacro">
     <!-- Include constants, materials, limb kinematics, & gazebo config -->
-    <xacro:include filename="$(find hector_assets)/models/xacro/const.xacro"/>
-    <xacro:include filename="$(find hector_assets)/models/xacro/materials.xacro"/>
-    <xacro:include filename="$(find hector_assets)/models/xacro/leg.xacro"/>
-    <xacro:include filename="$(find hector_assets)/models/xacro/arm.xacro"/>
+    <xacro:include filename="$(find hector_gazebo)/assets/models/xacro/const.xacro"/>
+    <xacro:include filename="$(find hector_gazebo)/assets/models/xacro/materials.xacro"/>
+    <xacro:include filename="$(find hector_gazebo)/assets/models/xacro/leg.xacro"/>
+    <xacro:include filename="$(find hector_gazebo)/assets/models/xacro/arm.xacro"/>
     <!-- Define the robot's trunk -->
-    <xacro:include filename="$(find hector_assets)/models/xacro/body.xacro"/>
+    <xacro:include filename="$(find hector_gazebo)/assets/models/xacro/body.xacro"/>
     <!-- Define the robot's legs -->
     <xacro:leg name="L" mirror="1" mirror_dae="False">
@@ -23,6 +23,6 @@
         <origin rpy="0 0 0" xyz="${hip_yaw_offset_x} ${-hip_yaw_offset_y} ${-hip_yaw_offset_z}"/>
     </xacro:arm>
-    <xacro:include filename="$(find hector_assets)/models/xacro/gazebo.xacro"/>
+    <xacro:include filename="$(find hector_gazebo)/assets/models/xacro/gazebo.xacro"/>
     <!-- Include the ros2_control plugins -->
-    <xacro:include filename="$(find hector_assets)/models/xacro/hardware.xacro"/>
+    <xacro:include filename="$(find hector_gazebo)/assets/models/xacro/hardware.xacro"/>
 </robot>
