Commit message: -finish new gazebo sim launch

File: src/hector_gazebo/assets/models/xacro/arm.xacro (robot description, xacro)
@@ -4,8 +4,8 @@
         <joint name="${name}_shoulder_yaw_joint" type="revolute">
             <xacro:if value="${(mirror_dae == True)}">
-            <origin rpy="0 0 0" xyz="0.0 0.047 0.1725"/>
+                <origin rpy="0 0 0" xyz="0.0 0.047 0.1725"/>
             </xacro:if>
             <xacro:if value="${(mirror_dae == False)}">
-            <origin rpy="0 0 0" xyz="0.0 -0.047 0.1725"/>
+                <origin rpy="0 0 0" xyz="0.0 -0.047 0.1725"/>
             </xacro:if>
             <parent link="trunk"/>
@@ -22,16 +22,16 @@
         <link name="${name}_shoulder_yaw_link">
             <visual>
-            <origin rpy="0 0 0" xyz="0 0 ${shoulder_yaw_offset_z}"/>
-            <xacro:if value="${(mirror_dae == True)}">
-            <geometry>
-                <mesh filename="file://$(find hector_gazebo)/assets/models/meshes/hector_arm/ShoulderYaw_L.stl" scale="1 1 1"/>
-            </geometry>
-            </xacro:if>
-            <xacro:if value="${(mirror_dae == False)}">
-            <geometry>
-                <mesh filename="file://$(find hector_gazebo)/assets/models/meshes/hector_arm/ShoulderYaw_R.stl" scale="1 1 1"/>
-            </geometry>
-            </xacro:if>
-            <material name="grey"/>
+                <origin rpy="0 0 0" xyz="0 0 ${shoulder_yaw_offset_z}"/>
+                <xacro:if value="${(mirror_dae == True)}">
+                    <geometry>
+                        <mesh filename="file://$(find hector_gazebo)/assets/models/meshes/hector_arm/ShoulderYaw_L.stl" scale="1 1 1"/>
+                    </geometry>
+                </xacro:if>
+                <xacro:if value="${(mirror_dae == False)}">
+                    <geometry>
+                        <mesh filename="file://$(find hector_gazebo)/assets/models/meshes/hector_arm/ShoulderYaw_R.stl" scale="1 1 1"/>
+                    </geometry>
+                </xacro:if>
+                <material name="grey"/>
             </visual>
             <collision>
@@ -42,18 +42,18 @@
             </collision>
             <inertial>
-                <origin rpy="0 0 0" xyz="${shoulder_yaw_com_x} ${shoulder_yaw_com_y*mirror} ${shoulder_yaw_com_z}"/>
+                <origin xyz="${shoulder_yaw_com_x} ${shoulder_yaw_com_y * mirror} ${shoulder_yaw_com_z}"
+                        rpy="${shoulder_yaw_rpy_r} ${shoulder_yaw_rpy_p} ${shoulder_yaw_rpy_y}"/>
                 <mass value="${shoulder_yaw_mass}"/>
-                <inertia
-                    ixx="${shoulder_yaw_ixx}" ixy="${shoulder_yaw_ixy*mirror}" ixz="${shoulder_yaw_ixz}"
-                    iyy="${shoulder_yaw_iyy}" iyz="${shoulder_yaw_iyz*mirror}"
-                    izz="${shoulder_yaw_izz}"/>
+                <inertia ixx="${shoulder_yaw_ixx}" ixy="0.0" ixz="0.0"
+                         iyy="${shoulder_yaw_iyy}" iyz="0.0"
+                         izz="${shoulder_yaw_izz}"/>
             </inertial>
         </link>
         <joint name="${name}_shoulder_pitch_joint" type="revolute">
             <xacro:if value="${(mirror_dae == True)}">
-            <origin rpy="0 0 0" xyz="0.0 0.045 -0.018"/>
+                <origin rpy="0 0 0" xyz="0.0 0.045 -0.018"/>
             </xacro:if>
             <xacro:if value="${(mirror_dae == False)}">
-            <origin rpy="0 0 0" xyz="0.0 -0.045 -0.018"/>
+                <origin rpy="0 0 0" xyz="0.0 -0.045 -0.018"/>
             </xacro:if>
             <parent link="${name}_shoulder_yaw_link"/>
@@ -65,18 +65,18 @@
         <link name="${name}_shoulder_pitch_link">
             <visual>
-            <origin rpy="0 0 0" xyz="0 0 0"/>
-            <xacro:if value="${(mirror_dae == True)}">
-            <geometry>
-                <mesh filename="file://$(find hector_gazebo)/assets/models/meshes/hector_arm/ShoulderPitch_L.stl" scale="1 1 1"/>
-            </geometry>
-            </xacro:if>
-            <xacro:if value="${(mirror_dae == False)}">
-            <geometry>
-                <mesh filename="file://$(find hector_gazebo)/assets/models/meshes/hector_arm/ShoulderPitch_R.stl" scale="1 1 1"/>
-            </geometry>
-            </xacro:if>
-            <material name="gold"/>
+                <origin rpy="0 0 0" xyz="0 0 0"/>
+                <xacro:if value="${(mirror_dae == True)}">
+                    <geometry>
+                        <mesh filename="file://$(find hector_gazebo)/assets/models/meshes/hector_arm/ShoulderPitch_L.stl" scale="1 1 1"/>
+                    </geometry>
+                </xacro:if>
+                <xacro:if value="${(mirror_dae == False)}">
+                    <geometry>
+                        <mesh filename="file://$(find hector_gazebo)/assets/models/meshes/hector_arm/ShoulderPitch_R.stl" scale="1 1 1"/>
+                    </geometry>
+                </xacro:if>
+                <material name="gold"/>
             </visual>
-           <collision>
+            <collision>
                 <origin rpy="0 ${PI/2.0} 0" xyz="0 0 ${-shoulder_pitch_length/2.0}"/>
                 <geometry>
@@ -88,15 +88,15 @@
                 <mass value="${shoulder_pitch_mass}"/>
                 <inertia
-                    ixx="${shoulder_pitch_ixx}" ixy="${shoulder_pitch_ixy*mirror}" ixz="${shoulder_pitch_ixz}"
-                    iyy="${shoulder_pitch_iyy}" iyz="${shoulder_pitch_iyz*mirror}"
-                    izz="${shoulder_pitch_izz}"/>
+                        ixx="${shoulder_pitch_ixx}" ixy="${shoulder_pitch_ixy*mirror}" ixz="${shoulder_pitch_ixz}"
+                        iyy="${shoulder_pitch_iyy}" iyz="${shoulder_pitch_iyz*mirror}"
+                        izz="${shoulder_pitch_izz}"/>
             </inertial>
         </link>
         <joint name="${name}_shoulder_roll_joint" type="revolute">
             <xacro:if value="${(mirror_dae == True)}">
-            <origin rpy="0 0 0" xyz="-0.0135 0.045 0.0"/>
+                <origin rpy="0 0 0" xyz="-0.0135 0.045 0.0"/>
             </xacro:if>
             <xacro:if value="${(mirror_dae == False)}">
-            <origin rpy="0 0 0" xyz="-0.0135 -0.045 0.0"/>
+                <origin rpy="0 0 0" xyz="-0.0135 -0.045 0.0"/>
             </xacro:if>
             <parent link="${name}_shoulder_pitch_link"/>
@@ -108,18 +108,18 @@
         <link name="${name}_shoulder_roll_link">
             <visual>
-            <origin rpy="0 0 0" xyz="0 0 0"/>
-            <xacro:if value="${(mirror_dae == True)}">
-            <geometry>
-                <mesh filename="file://$(find hector_gazebo)/assets/models/meshes/hector_arm/UpperArmRoll_L.stl" scale="1 1 1"/>
-            </geometry>
-            </xacro:if>
-            <xacro:if value="${(mirror_dae == False)}">
-            <geometry>
-                <mesh filename="file://$(find hector_gazebo)/assets/models/meshes/hector_arm/UpperArmRoll_R.stl" scale="1 1 1"/>
-            </geometry>
-            </xacro:if>
-            <material name="grey"/>
+                <origin rpy="0 0 0" xyz="0 0 0"/>
+                <xacro:if value="${(mirror_dae == True)}">
+                    <geometry>
+                        <mesh filename="file://$(find hector_gazebo)/assets/models/meshes/hector_arm/UpperArmRoll_L.stl" scale="1 1 1"/>
+                    </geometry>
+                </xacro:if>
+                <xacro:if value="${(mirror_dae == False)}">
+                    <geometry>
+                        <mesh filename="file://$(find hector_gazebo)/assets/models/meshes/hector_arm/UpperArmRoll_R.stl" scale="1 1 1"/>
+                    </geometry>
+                </xacro:if>
+                <material name="grey"/>
             </visual>
-           <collision>
+            <collision>
                 <origin rpy="0 ${PI/2.0} 0" xyz="${shoulder_roll_offset_x} 0 ${-shoulder_roll_length/2.0}"/>
                 <geometry>
@@ -131,7 +131,7 @@
                 <mass value="${shoulder_roll_mass}"/>
                 <inertia
-                    ixx="${shoulder_roll_ixx}" ixy="${shoulder_roll_ixy*mirror}" ixz="${shoulder_roll_ixz}"
-                    iyy="${shoulder_roll_iyy}" iyz="${shoulder_roll_iyz*mirror}"
-                    izz="${shoulder_roll_izz}"/>
+                        ixx="${shoulder_roll_ixx}" ixy="${shoulder_roll_ixy*mirror}" ixz="${shoulder_roll_ixz}"
+                        iyy="${shoulder_roll_iyy}" iyz="${shoulder_roll_iyz*mirror}"
+                        izz="${shoulder_roll_izz}"/>
             </inertial>
         </link>
@@ -146,9 +146,9 @@
         <link name="${name}_elbow_link">
             <visual>
-            <origin rpy="0 0 0" xyz="0 0 0"/>
-            <geometry>
-                <mesh filename="file://$(find hector_gazebo)/assets/models/meshes/hector_arm/ForeArmPitch.stl" scale="1 1 1"/>
-            </geometry>
-            <material name="grey"/>
+                <origin rpy="0 0 0" xyz="0 0 0"/>
+                <geometry>
+                    <mesh filename="file://$(find hector_gazebo)/assets/models/meshes/hector_arm/ForeArmPitch.stl" scale="1 1 1"/>
+                </geometry>
+                <material name="grey"/>
             </visual>
             <collision>
@@ -162,7 +162,7 @@
                 <mass value="${elbow_mass}"/>
                 <inertia
-                    ixx="${elbow_ixx}" ixy="${elbow_ixy}" ixz="${elbow_ixz}"
-                    iyy="${elbow_iyy}" iyz="${elbow_iyz}"
-                    izz="${elbow_izz}"/>
+                        ixx="${elbow_ixx}" ixy="${elbow_ixy}" ixz="${elbow_ixz}"
+                        iyy="${elbow_iyy}" iyz="${elbow_iyz}"
+                        izz="${elbow_izz}"/>
             </inertial>
         </link>
@@ -174,9 +174,9 @@
         <link name="${name}_arm_EE_link">
             <visual>
-            <origin rpy="0 0 0" xyz="0 0 0"/>
-            <geometry>
-                <sphere radius="0.01"/>
-            </geometry>
-            <material name="grey"/>
+                <origin rpy="0 0 0" xyz="0 0 0"/>
+                <geometry>
+                    <sphere radius="0.01"/>
+                </geometry>
+                <material name="grey"/>
             </visual>
             <inertial>
@@ -184,7 +184,7 @@
                 <mass value="0.0001"/>
                 <inertia
-                    ixx="0.0000001" ixy="0.0000001" ixz="0.0000001"
-                    iyy="0.0000001" iyz="0.0000001"
-                    izz="0.0000001"/>
+                        ixx="0.0000001" ixy="0.0" ixz="0.0"
+                        iyy="0.0000001" iyz="0.0"
+                        izz="0.0000001"/>
             </inertial>
         </link>

File: src/hector_gazebo/assets/models/xacro/const.xacro (robot description, xacro)
@@ -238,14 +238,13 @@
     <xacro:property name="shoulder_yaw_length" value="0.08"/>
     <!-- inertial -->
-    <!-- <xacro:property name="shoulder_yaw_mass" value="1.096"/> -->
     <xacro:property name="shoulder_yaw_mass" value="0.4356"/>
     <xacro:property name="shoulder_yaw_com_x" value="0.00071"/>
     <xacro:property name="shoulder_yaw_com_y" value="0.02838"/>
     <xacro:property name="shoulder_yaw_com_z" value="0.04835"/>
-    <xacro:property name="shoulder_yaw_ixx" value="0.00035"/>
-    <xacro:property name="shoulder_yaw_ixy" value="0.0"/>
-    <xacro:property name="shoulder_yaw_ixz" value="0.00002"/>
-    <xacro:property name="shoulder_yaw_iyy" value="0.00043"/>
-    <xacro:property name="shoulder_yaw_iyz" value="0.00063"/>
+    <xacro:property name="shoulder_yaw_rpy_r" value="0.0"/>
+    <xacro:property name="shoulder_yaw_rpy_p" value="0.0"/>
+    <xacro:property name="shoulder_yaw_rpy_y" value="1.570796"/>
+    <xacro:property name="shoulder_yaw_ixx" value="0.00043"/>
+    <xacro:property name="shoulder_yaw_iyy" value="0.00035"/>
     <xacro:property name="shoulder_yaw_izz" value="0.00027"/>
     <!-- shoulder_pitch -->

File: src/hector_gazebo/assets/models/xacro/gazebo.xacro (robot description, xacro)
@@ -1,232 +1,117 @@
 <?xml version="1.0"?>
-<robot>
-    <!-- Show the trajectory of trunk center. -->
-    <gazebo>
-        <plugin name="3dplot" filename="libLinkPlot3DPlugin.so">
-            <frequency>10</frequency>
-            <plot>
-                <link>trunk</link>
-                <pose>0 0 0 0 0 0</pose>
-                <material>Gazebo/Gold</material>
-            </plot>
-        </plugin>
-    </gazebo>
-    <gazebo>
-        <plugin name="3dplot" filename="libLinkPlot3DPlugin.so">
-          <frequency>100</frequency>
-          <plot>
-            <link>R_EE_link</link>
-            <pose>0 0 0 0 0 0</pose>
-            <material>Gazebo/Gold</material>
-          </plot>
-        </plugin>
-    </gazebo>
-      <!-- <gazebo>
-        <plugin name="3dplot" filename="libLinkPlot3DPlugin.so">
-          <frequency>100</frequency>
-          <plot>
-            <link>R_elbow_link</link>
-            <pose>0 0 0 0 0 0</pose>
-            <material>Gazebo/Gold</material>
-          </plot>
-        </plugin>
-      </gazebo> -->
+<robot xmlns:xacro="http://www.ros.org/wiki/xacro">
     <gazebo reference="imu_link">
-        <gravity>true</gravity>
         <sensor name="imu_sensor" type="imu">
             <always_on>true</always_on>
             <update_rate>1000</update_rate>
             <visualize>true</visualize>
-            <topic>__default_topic__</topic>
-            <plugin filename="libgazebo_ros_imu_sensor.so" name="imu_plugin">
-                <topicName>trunk_imu</topicName>
-                <bodyName>imu_link</bodyName>
-                <updateRateHZ>1000.0</updateRateHZ>
-                <gaussianNoise>0.00</gaussianNoise>
-                <xyzOffset>0 0 0</xyzOffset>
-                <rpyOffset>0 0 0</rpyOffset>
-                <frameName>imu_link</frameName>
-            </plugin>
-            <pose>0 0 0 0 0 0</pose>
+            <imu>
+                <angular_velocity>
+                    <x>
+                        <noise type="gaussian">
+                            <mean>0.0</mean>
+                            <stddev>0.0002</stddev> <bias_mean>0.0000075</bias_mean>
+                            <bias_stddev>0.0000008</bias_stddev>
+                        </noise>
+                    </x>
+                    <y>
+                        <noise type="gaussian">
+                            <mean>0.0</mean>
+                            <stddev>0.0002</stddev> <bias_mean>0.0000075</bias_mean>
+                            <bias_stddev>0.0000008</bias_stddev>
+                        </noise>
+                    </y>
+                    <z>
+                        <noise type="gaussian">
+                            <mean>0.0</mean>
+                            <stddev>0.0002</stddev> <bias_mean>0.0000075</bias_mean>
+                            <bias_stddev>0.0000008</bias_stddev>
+                        </noise>
+                    </z>
+                </angular_velocity>
+                <linear_acceleration>
+                    <x>
+                        <noise type="gaussian">
+                            <mean>0.0</mean>
+                            <stddev>0.017</stddev> <bias_mean>0.1</bias_mean>
+                            <bias_stddev>0.001</bias_stddev>
+                        </noise>
+                    </x>
+                    <y>
+                        <noise type="gaussian">
+                            <mean>0.0</mean>
+                            <stddev>0.017</stddev> <bias_mean>0.1</bias_mean>
+                            <bias_stddev>0.001</bias_stddev>
+                        </noise>
+                    </y>
+                    <z>
+                        <noise type="gaussian">
+                            <mean>0.0</mean>
+                            <stddev>0.017</stddev> <bias_mean>0.1</bias_mean>
+                            <bias_stddev>0.001</bias_stddev>
+                        </noise>
+                    </z>
+                </linear_acceleration>
+            </imu>
+            <plugin name="gz::sim::systems::Imu" filename="gz-sim-imu-system"/>
         </sensor>
     </gazebo>
     <gazebo reference="base">
-        <material>Gazebo/Green</material>
-        <turnGravityOff>false</turnGravityOff>
     </gazebo>
     <gazebo reference="trunk">
-        <mu1>0.2</mu1>
-        <mu2>0.2</mu2>
-        <material>Gazebo/DarkGrey</material>
     </gazebo>
-     <gazebo reference="trunkcol">
-        <mu1>0.2</mu1>
-        <mu2>0.2</mu2>
+    <gazebo reference="trunkcol">
     </gazebo>
     <gazebo reference="stick_link">
-        <mu1>0.2</mu1>
-        <mu2>0.2</mu2>
-        <material>Gazebo/White</material>
     </gazebo>
     <gazebo reference="imu_link">
-        <mu1>1</mu1>
-        <mu2>1</mu2>
-        <material>Gazebo/Black</material>
     </gazebo>
-    <!-- L leg -->
     <gazebo reference="L_hip_yaw_link">
-        <mu1>1</mu1>
-        <mu2>1</mu2>
-        <kp  value="100000.0"/>
-        <kd  value="1000.0"/>
-        <material>Gazebo/Grey</material>
     </gazebo>
     <gazebo reference="L_hip_roll_link">
-        <mu1>1</mu1>
-        <mu2>1</mu2>
-        <kp  value="100000.0"/>
-        <kd  value="1000.0"/>
-        <material>Gazebo/Gold</material>
     </gazebo>
     <gazebo reference="L_hip_pitch_link">
-        <mu1>1</mu1>
-        <mu2>1</mu2>
-        <kp  value="100000.0"/>
-        <kd  value="1000.0"/>
-        <self_collide>0</self_collide>
-        <material>Gazebo/Grey</material>
     </gazebo>
     <gazebo reference="L_knee_link">
-        <mu1>1</mu1>
-        <mu2>1</mu2>
-        <kp  value="100000.0"/>
-        <kd  value="1000.0"/>
-        <self_collide>0</self_collide>
-        <material>Gazebo/Grey</material>
     </gazebo>
     <gazebo reference="L_ankle_link">
-        <mu1>3</mu1>
-        <mu2>3</mu2>
-        <kp  value="1000000.0"/>
-        <kd  value="1000.0"/>
-        <self_collide>0</self_collide>
-        <material>Gazebo/Grey</material>
     </gazebo>
-    <!--R leg -->
     <gazebo reference="R_hip_yaw_link">
-        <mu1>1</mu1>
-        <mu2>1</mu2>
-        <kp  value="100000.0"/>
-        <kd  value="1000.0"/>
-        <material>Gazebo/Grey</material>
     </gazebo>
     <gazebo reference="R_hip_roll_link">
-        <mu1>1</mu1>
-        <mu2>1</mu2>
-        <kp  value="100000.0"/>
-        <kd  value="1000.0"/>
-        <material>Gazebo/Gold</material>
     </gazebo>
     <gazebo reference="R_hip_pitch_link">
-        <mu1>1</mu1>
-        <mu2>1</mu2>
-        <kp  value="100000.0"/>
-        <kd  value="1000.0"/>
-        <self_collide>0</self_collide>
-        <material>Gazebo/Grey</material>
     </gazebo>
     <gazebo reference="R_knee_link">
-        <mu1>1</mu1>
-        <mu2>1</mu2>
-        <kp  value="100000.0"/>
-        <kd  value="1000.0"/>
-        <self_collide>0</self_collide>
-        <material>Gazebo/Grey</material>
     </gazebo>
     <gazebo reference="R_ankle_link">
-        <mu1>3</mu1>
-        <mu2>3</mu2>
-        <kp  value="1000000.0"/>
-        <kd  value="1000.0"/>
-        <self_collide>0</self_collide>
-        <material>Gazebo/Grey</material>
     </gazebo>
-    <!-- L arm -->
     <gazebo reference="L_shoulder_yaw_link">
-        <mu1>1</mu1>
-        <mu2>1</mu2>
-        <kp  value="100000.0"/>
-        <kd  value="1000.0"/>
-        <material>Gazebo/Gold</material>
     </gazebo>
     <gazebo reference="L_shoulder_pitch_link">
-        <mu1>1</mu1>
-        <mu2>1</mu2>
-        <kp  value="100000.0"/>
-        <kd  value="1000.0"/>
-        <material>Gazebo/Grey</material>
     </gazebo>
     <gazebo reference="L_shoulder_roll_link">
-        <mu1>1</mu1>
-        <mu2>1</mu2>
-        <kp  value="100000.0"/>
-        <kd  value="1000.0"/>
-        <material>Gazebo/Grey</material>
     </gazebo>
     <gazebo reference="L_elbow_link">
-        <mu1>3</mu1>
-        <mu2>3</mu2>
-        <kp  value="1000000.0"/>
-        <kd  value="1000.0"/>
-        <material>Gazebo/Grey</material>
     </gazebo>
-    <!-- R arm -->
     <gazebo reference="R_shoulder_yaw_link">
-        <mu1>1</mu1>
-        <mu2>1</mu2>
-        <kp  value="100000.0"/>
-        <kd  value="1000.0"/>
-        <material>Gazebo/Gold</material>
     </gazebo>
     <gazebo reference="R_shoulder_pitch_link">
-        <mu1>1</mu1>
-        <mu2>1</mu2>
-        <kp  value="100000.0"/>
-        <kd  value="1000.0"/>
-        <material>Gazebo/Grey</material>
     </gazebo>
     <gazebo reference="R_shoulder_roll_link">
-        <mu1>1</mu1>
-        <mu2>1</mu2>
-        <kp  value="100000.0"/>
-        <kd  value="1000.0"/>
-        <material>Gazebo/Grey</material>
     </gazebo>
     <gazebo reference="R_elbow_link">
-        <mu1>3</mu1>
-        <mu2>3</mu2>
-        <kp  value="1000000.0"/>
-        <kd  value="1000.0"/>
-        <material>Gazebo/Grey</material>
     </gazebo>
-    <!-- head_link -->
     <gazebo reference="head_link">
-        <material>Gazebo/Grey</material>
     </gazebo>
-    <!--NUC link  -->
     <gazebo reference="nuc_link">
-        <material>Gazebo/DarkGrey</material>
     </gazebo>
     <gazebo reference="L_arm_EE_link">
-        <material>Gazebo/Gold</material>
     </gazebo>
     <gazebo reference="R_arm_EE_link">
-        <material>Gazebo/Gold</material>
     </gazebo>
     <gazebo reference="L_leg_EE_link">
-        <material>Gazebo/Gold</material>
     </gazebo>
     <gazebo reference="R_leg_EE_link">
-        <material>Gazebo/Gold</material>
     </gazebo>
 </robot>
