Commit message: - Implement basic framework for the Hector Gazebo Fortress system plugin. - Perform initial modifications to robot asset Xacro files for compatibility.

File: src/hector_gazebo/assets/models/xacro/gazebo.xacro (robot description, xacro)
@@ -1,4 +1,32 @@
 <?xml version="1.0"?>
 <robot xmlns:xacro="http://www.ros.org/wiki/xacro">
+    <gazebo reference="base_link">
+        <plugin
+                filename="libhector_gazebo_fortress_plugin.so"
+                name="hector_gazebo_plugins::HectorGazeboFortressPlugin">
+            <joint_name>L_hip_yaw_joint</joint_name>
+            <joint_name>L_hip_roll_joint</joint_name>
+            <joint_name>L_hip_pitch_joint</joint_name>
+            <joint_name>L_knee_joint</joint_name>
+            <joint_name>L_ankle_joint</joint_name>
+            <joint_name>R_hip_yaw_joint</joint_name>
+            <joint_name>R_hip_roll_joint</joint_name>
+            <joint_name>R_hip_pitch_joint</joint_name>
+            <joint_name>R_knee_joint</joint_name>
+            <joint_name>R_ankle_joint</joint_name>
+            <joint_name>L_shoulder_yaw_joint</joint_name>
+            <joint_name>L_shoulder_pitch_joint</joint_name>
+            <joint_name>L_shoulder_roll_joint</joint_name>
+            <joint_name>L_elbow_joint</joint_name>
+            <joint_name>R_shoulder_yaw_joint</joint_name>
+            <joint_name>R_shoulder_pitch_joint</joint_name>
+            <joint_name>R_shoulder_roll_joint</joint_name>
+            <joint_name>R_elbow_joint</joint_name>
+            <base_link_name>base_link</base_link_name>
+            <ign_imu_topic>/imu</ign_imu_topic>
+            <ign_left_contact_topic>/l_contact</ign_left_contact_topic>
+            <ign_right_contact_topic>/r_contact</ign_right_contact_topic>
+        </plugin>
+    </gazebo>
     <gazebo reference="imu_link">
         <sensor name="imu_sensor" type="imu">
@@ -6,4 +34,5 @@
             <update_rate>1000</update_rate>
             <visualize>true</visualize>
+            <topic>/imu</topic>
             <imu>
                 <angular_velocity>
@@ -54,5 +83,31 @@
                 </linear_acceleration>
             </imu>
-            <plugin name="gz::sim::systems::Imu" filename="gz-sim-imu-system"/>
+            <plugin filename="libignition-gazebo-imu-system.so"
+                    name="ignition::gazebo::systems::Imu">
+            </plugin>
+        </sensor>
+    </gazebo>
+    <gazebo reference="L_ankle_link">
+        <sensor name="left_foot_contact" type="contact">
+            <always_on>true</always_on>
+            <update_rate>50</update_rate>
+            <contact>
+                <collision>L_foot_collision</collision>
+            </contact>
+            <topic>/l_contact</topic>
+            <plugin filename="libignition-gazebo-contact-system.so" name="ignition::gazebo::systems::Contact">
+            </plugin>
+        </sensor>
+    </gazebo>
+    <gazebo reference="R_ankle_link">
+        <sensor name="right_foot_contact" type="contact">
+            <always_on>true</always_on>
+            <update_rate>50</update_rate>
+            <contact>
+                <collision>R_foot_collision</collision>
+            </contact>
+            <topic>/r_contact</topic>
+            <plugin filename="libignition-gazebo-contact-system.so" name="ignition::gazebo::systems::Contact">
+            </plugin>
         </sensor>
     </gazebo>

File: src/hector_gazebo/assets/models/xacro/leg.xacro (robot description, xacro)
@@ -1,5 +1,4 @@
 <?xml version="1.0"?>
 <robot xmlns:xacro="http://www.ros.org/wiki/xacro">
-    <!-- <xacro:include filename="$(find hector_gazebo)/assets/models/xacro/transmission.xacro"/> -->
     <xacro:macro name="leg" params="name mirror mirror_dae  *origin">
         <joint name="${name}_hip_yaw_joint" type="revolute">
@@ -282,5 +281,5 @@
                 <material name="grey"/>
             </visual>
-            <collision>
+            <collision name="${name}_foot_collision">
                 <origin rpy="0 0 0" xyz="${ankle_x} ${ankle_y*mirror} ${ankle_z}"/>
                 <geometry>

File: src/hector_gazebo/assets/models/xacro/robot.xacro (robot description, xacro)
@@ -25,4 +25,4 @@
     <xacro:include filename="$(find hector_gazebo)/assets/models/xacro/gazebo.xacro"/>
     <!-- Include the ros2_control plugins -->
-    <xacro:include filename="$(find hector_gazebo)/assets/models/xacro/hardware.xacro"/>
+<!--    <xacro:include filename="$(find hector_gazebo)/assets/models/xacro/hardware.xacro"/>-->
 </robot>
